Commit message: Robot moves

File: data/urdf/so100.urdf (robot description, URDF)
Before this commit: robot so100_minimal, 6 links, 5 joints
Joints:
- joint forearm_joint: origin xyz=0.112 0 -0.028 rpy=0 0 0 -> xyz=0.112 0 -0.028 rpy=0 1.5708 0
- joint humerus_joint: axis 0 -1 0 -> 0 1 0; origin xyz=0.031 0 0.072 rpy=0 0 0 -> xyz=0.031 0 0.072 rpy=0 -1.5708 0

File: data/urdf/so101.urdf (robot description, URDF)
Before this commit: robot so101_minimal, 6 links, 5 joints
Joints:
- joint humerus_joint: axis 0 -1 0 -> 0 1 0
